Commit message: modifided gazebo controller

File: simpleDog/urdf/robot.urdf (robot description, URDF)
Before this commit: robot simpledog, 19 links, 18 joints
Links:
- link lh_foot_Link: geometry collision mesh filename=package://simpledog/meshes/rh_foot_Link.STL; visual mesh filename=package://simpledog/meshes/rh_foot_Link.STL
- link rh_foot_Link: geometry collision mesh filename=package://simpledog/meshes/lh_foot_Link.STL; visual mesh filename=package://simpledog/meshes/lh_foot_Link.STL
Joints:
- joint front_left_1_joint: limit lower=-3.0 upper=3.0 effort=100 velocity=10 -> lower=-3.0 upper=3.0 effort=300 velocity=10
- joint front_left_2_joint: limit lower=-3.0 upper=3.0 effort=100 velocity=10 -> lower=-3.0 upper=3.0 effort=300 velocity=10
- joint front_left_3_joint: limit lower=-3.0 upper=3.0 effort=100 velocity=10 -> lower=-3.0 upper=3.0 effort=300 velocity=10
- joint front_right_1_joint: limit lower=-3.0 upper=3.0 effort=100 velocity=10 -> lower=-3.0 upper=3.0 effort=300 velocity=10
- joint front_right_2_joint: limit lower=-3.0 upper=3.0 effort=100 velocity=10 -> lower=-3.0 upper=3.0 effort=300 velocity=10
- joint front_right_3_joint: limit lower=-3.0 upper=3.0 effort=100 velocity=10 -> lower=-3.0 upper=3.0 effort=300 velocity=10
- joint lh_foot_joint: origin xyz=0.24968 0.00033355 -0.015 rpy=0 0 0 -> xyz=0.24742286767759 0.000379574544590811 -0.015 rpy=0 0 0; parent rear_right_3_Link -> rear_left_3_Link
- joint rear_left_1_joint: limit lower=-3.0 upper=3.0 effort=100 velocity=10 -> lower=-3.0 upper=3.0 effort=300 velocity=10
- joint rear_left_2_joint: limit lower=-3.0 upper=3.0 effort=100 velocity=10 -> lower=-3.0 upper=3.0 effort=300 velocity=10
- joint rear_left_3_joint: limit lower=-3.0 upper=3.0 effort=100 velocity=10 -> lower=-3.0 upper=3.0 effort=300 velocity=10
- joint rear_right_1_joint: limit lower=-3.0 upper=3.0 effort=100 velocity=10 -> lower=-3.0 upper=3.0 effort=300 velocity=10
- joint rear_right_2_joint: limit lower=-3.0 upper=3.0 effort=100 velocity=10 -> lower=-3.0 upper=3.0 effort=300 velocity=10
- joint rear_right_3_joint: limit lower=-3.0 upper=3.0 effort=100 velocity=10 -> lower=-3.0 upper=3.0 effort=300 velocity=10
- joint rh_foot_joint: origin xyz=0.24742286767759 0.000379574544590811 -0.015 rpy=0 0 0 -> xyz=0.24968 0.00033355 -0.015 rpy=0 0 0; parent rear_left_3_Link -> rear_right_3_Link

File: simpleDog/urdf/simpledog.urdf.xacro (robot description, xacro)
@@ -33,6 +33,6 @@
 <xacro:simpledog_foot_sensors foot_prefix="lf_foot" joint_prefix="front_left_3_"> </xacro:simpledog_foot_sensors>
 <xacro:simpledog_foot_sensors foot_prefix="rf_foot" joint_prefix="front_right_3_"> </xacro:simpledog_foot_sensors>
-<xacro:simpledog_foot_sensors foot_prefix="rh_foot" joint_prefix="rear_left_3_"> </xacro:simpledog_foot_sensors>
-<xacro:simpledog_foot_sensors foot_prefix="lh_foot" joint_prefix="rear_right_3_"> </xacro:simpledog_foot_sensors>
+<xacro:simpledog_foot_sensors foot_prefix="rh_foot" joint_prefix="rear_right_3_"> </xacro:simpledog_foot_sensors>
+<xacro:simpledog_foot_sensors foot_prefix="lh_foot" joint_prefix="rear_left_3_"> </xacro:simpledog_foot_sensors>
 <link
     name="base_link">
@@ -42,5 +42,5 @@
         rpy="0 0 0" />
       <mass
-        value="15.238" />
+        value="22.5" />
       <inertia
         ixx="0.74932"
@@ -128,5 +128,5 @@
       xyz="0 0 1" />
       <limit
-      effort="100"
+      effort="300"
       velocity="10"
       lower="-3.0"
@@ -186,5 +186,5 @@
       xyz="0 0 1" />
       <limit
-      effort="100"
+      effort="300"
       velocity="10"
       lower="-3.0"
@@ -244,5 +244,5 @@
       xyz="0 0 1" />
       <limit
-      effort="100"
+      effort="300"
       velocity="10"
       lower="-3.0"
@@ -355,5 +355,5 @@
       xyz="0 0 1" />
       <limit
-      effort="100"
+      effort="300"
       velocity="10"
       lower="-3.0"
@@ -413,5 +413,5 @@
       xyz="0 0 1" />
       <limit
-      effort="100"
+      effort="300"
       velocity="10"
       lower="-3.0"
@@ -471,5 +471,5 @@
       xyz="0 0 1" />
       <limit
-      effort="100"
+      effort="300"
       velocity="10"
       lower="-3.0"
@@ -582,5 +582,5 @@
       xyz="0 0 1" />
       <limit
-      effort="100"
+      effort="300"
       velocity="10"
       lower="-3.0"
@@ -640,5 +640,5 @@
       xyz="0 0 1" />
       <limit
-      effort="100"
+      effort="300"
       velocity="10"
       lower="-3.0"
@@ -698,11 +698,11 @@
       xyz="0 0 1" />
       <limit
-      effort="100"
-      velocity="10"
-      lower="-3.0"
-      upper="3.0"/>
-  </joint>
-  <link
-    name="rh_foot_Link">
+      effort="300"
+      velocity="10"
+      lower="-3.0"
+      upper="3.0"/>
+  </joint>
+  <link
+    name="lh_foot_Link">
     <inertial>
       <origin
@@ -744,5 +744,5 @@
   </link>
   <joint
-    name="rh_foot_joint"
+    name="lh_foot_joint"
     type="fixed">
     <origin
@@ -752,5 +752,5 @@
       link="rear_left_3_Link" />
     <child
-      link="rh_foot_Link" />
+      link="lh_foot_Link" />
     <axis
       xyz="0 0 0" />
@@ -809,5 +809,5 @@
       xyz="0 0 1" />
       <limit
-      effort="100"
+      effort="300"
       velocity="10"
       lower="-3.0"
@@ -867,5 +867,5 @@
       xyz="0 0 1" />
       <limit
-      effort="100"
+      effort="300"
       velocity="10"
       lower="-3.0"
@@ -925,11 +925,11 @@
       xyz="0 0 1" />
       <limit
-      effort="100"
-      velocity="10"
-      lower="-3.0"
-      upper="3.0"/>
-  </joint>
-  <link
-    name="lh_foot_Link">
+      effort="300"
+      velocity="10"
+      lower="-3.0"
+      upper="3.0"/>
+  </joint>
+  <link
+    name="rh_foot_Link">
     <inertial>
       <origin
@@ -971,5 +971,5 @@
   </link>
   <joint
-    name="lh_foot_joint"
+    name="rh_foot_joint"
     type="fixed">
     <origin
@@ -979,5 +979,5 @@
       link="rear_right_3_Link" />
     <child
-      link="lh_foot_Link" />
+      link="rh_foot_Link" />
     <axis
       xyz="0 0 0" />

File: simpleDog/urdf/simpledog_gazebo.urdf.xacro (robot description, xacro)
@@ -16,6 +16,7 @@
 <!--load the gazebo rosz-control plug in-->
 <gazebo>
-  <plugin name="gazebo_ros_control" filename="libgazebo_ros_control.so">
+  <plugin name="balance_controller" filename="librobot_state_gazebo_ros_control_plugin.so">
     <robotNamespace>$(arg robot_namespace)</robotNamespace>
+    <robotSimType>balance_controller/SimRobotStateHardwareInterface</robotSimType>
   </plugin>
 </gazebo>
