Commit message: fix contact sensor

File: simpleDog/urdf/simpledog.urdf.xacro (robot description, xacro)
@@ -8,9 +8,10 @@
   <xacro:include filename="$(find simpledog)/urdf/joint_gazebo.urdf.xacro" />
   <xacro:include filename="$(find simpledog)/urdf/kinect.urdf.xacro"/>
+  <xacro:include filename="$(find simpledog)/urdf/foot_sensor_gazebo.urdf.xacro" />
 <!--load kinect urdf-->
 <xacro:if value="$(arg kinect_enabled)">
   <xacro:kinect_camera prefix="camera" robot_namespace="$(arg robot_namespace)"/>
   <joint name="kinect_frame_joint" type="fixed">
-    <origin xyz="-0.3 0 0.1" rpy="0 0.18 3.14159" />
+    <origin xyz="0.3 0 0.1" rpy="0 0.18 0" />
     <parent link="base_link"/>
     <child link="camera_link"/>
@@ -30,9 +31,13 @@
 <xacro:simpledog_joint joint_prefix="rear_left_2_"> </xacro:simpledog_joint>
 <xacro:simpledog_joint joint_prefix="rear_left_3_"> </xacro:simpledog_joint>
-  <link
+<xacro:simpledog_foot_sensors foot_prefix="lf_foot" joint_prefix="front_left_3_"> </xacro:simpledog_foot_sensors>
+<xacro:simpledog_foot_sensors foot_prefix="rf_foot" joint_prefix="front_right_3_"> </xacro:simpledog_foot_sensors>
+<xacro:simpledog_foot_sensors foot_prefix="rh_foot" joint_prefix="rear_left_3_"> </xacro:simpledog_foot_sensors>
+<xacro:simpledog_foot_sensors foot_prefix="lh_foot" joint_prefix="rear_right_3_"> </xacro:simpledog_foot_sensors>
+<link
     name="base_link">
     <inertial>
       <origin
-        xyz="-2.919E-17 4.8611E-17 9.4163E-19"
+        xyz="2.919E-17 -4.8141E-17 9.4163E-19"
         rpy="0 0 0" />
       <mass
@@ -41,7 +46,7 @@
         ixx="0.74932"
         ixy="-1.2062E-17"
-        ixz="-1.9781E-17"
+        ixz="-2.0602E-16"
         iyy="2.3017"
-        iyz="7.9134E-17"
+        iyz="-3.8366E-17"
         izz="2.9675" />
     </inertial>
@@ -74,14 +79,14 @@
     <inertial>
       <origin
-        xyz="-0.012793 -1.5357E-15 0.04"
+        xyz="1.7015E-17 0.012793 -0.00023552"
         rpy="0 0 0" />
       <mass
         value="1.1709" />
       <inertia
-        ixx="0.0013167"
-        ixy="-4.8862E-17"
-        ixz="7.6795E-20"
-        iyy="0.001719"
-        iyz="-1.6433E-19"
+        ixx="0.001719"
+        ixy="2.9302E-20"
+        ixz="-1.6433E-19"
+        iyy="0.0013167"
+        iyz="-7.6795E-20"
         izz="0.0021511" />
     </inertial>
@@ -114,6 +119,6 @@
     type="revolute">
     <origin
-      xyz="-0.36 -0.175 0"
-      rpy="-1.5708 0 1.5708" />
+      xyz="0.400 0.175 0"
+      rpy="1.57079632679453 1.57051603921301 1.57079632679453" />
     <parent
       link="base_link" />
@@ -122,12 +127,9 @@
     <axis
       xyz="0 0 1" />
-    <sensor name="force_torque" type="force_torque">
-        <update_rate>30</update_rate>
-    </sensor>
-      <limit
-        effort="100"
-        velocity="10"
-        lower="-3.0"
-        upper="3.0"/>
+      <limit
+      effort="100"
+      velocity="10"
+      lower="-3.0"
+      upper="3.0"/>
   </joint>
   <link
@@ -135,15 +137,15 @@
     <inertial>
       <origin
-        xyz="0.025099 2.8253E-06 -0.11431"
+        xyz="0.11439 0.00028184 0.05942"
         rpy="0 0 0" />
       <mass
         value="1.3902" />
       <inertia
-        ixx="0.028484"
-        ixy="2.4654E-16"
-        ixz="1.2624E-14"
+        ixx="0.0030209"
+        ixy="-5.6504E-20"
+        ixz="2.8413E-18"
         iyy="0.026875"
-        iyz="5.6397E-18"
-        izz="0.0030209" />
+        iyz="1.5349E-06"
+        izz="0.028484" />
     </inertial>
     <visual>
@@ -175,6 +177,6 @@
     type="revolute">
     <origin
-      xyz="-0.034321 0 0.04"
-      rpy="-1.5708 0 3.1416" />
+      xyz="0 0 0"
+      rpy="-1.5708 0 0" />
     <parent
       link="front_left_1_Link" />
@@ -182,10 +184,10 @@
       link="front_left_2_Link" />
     <axis
-      xyz="1 0 0" />
-      <limit
-        effort="100"
-        velocity="10"
-        lower="-3.0"
-        upper="3.0"/>
+      xyz="0 0 1" />
+      <limit
+      effort="100"
+      velocity="10"
+      lower="-3.0"
+      upper="3.0"/>
   </joint>
   <link
@@ -193,72 +195,352 @@
     <inertial>
       <origin
-        xyz="-0.043355 -1.0168E-05 -0.087821"
+        xyz="0.087825 1.529E-05 -0.016708"
         rpy="0 0 0" />
       <mass
         value="1.3523" />
       <inertia
-        ixx="0.0093381"
-        ixy="-2.3773E-08"
+        ixx="0.00053032"
+        ixy="-8.5291E-07"
+        ixz="-0.00020744"
+        iyy="0.0091429"
+        iyz="-8.3738E-08"
+        izz="0.009338" />
+    </inertial>
+    <visual>
+      <origin
+        xyz="0 0 0"
+        rpy="0 0 0" />
+      <geometry>
+        <mesh
+          filename="package://simpledog/meshes/front_left_3_Link.STL" />
+      </geometry>
+      <material
+        name="">
+        <color
+          rgba="0.89804 0.91765 0.92941 1" />
+      </material>
+    </visual>
+    <collision>
+      <origin
+        xyz="0 0 0"
+        rpy="0 0 0" />
+      <geometry>
+        <mesh
+          filename="package://simpledog/meshes/front_left_3_Link.STL" />
+      </geometry>
+    </collision>
+  </link>
+  <joint
+    name="front_left_3_joint"
+    type="revolute">
+    <origin
+      xyz="0.250069171339977 0.000334332414087979 0.11441948932032"
+      rpy="0 0 0" />
+    <parent
+      link="front_left_2_Link" />
+    <child
+      link="front_left_3_Link" />
+    <axis
+      xyz="0 0 1" />
+      <limit
+      effort="100"
+      velocity="10"
+      lower="-3.0"
+      upper="3.0"/>
+  </joint>
+  <link
+    name="lf_foot_Link">
+    <inertial>
+      <origin
+        xyz="0.0178251114319979 0 0"
+        rpy="0 0 0" />
+      <mass
+        value="0.0556193699314689" />
+      <inertia
+        ixx="1.65498601680364E-05"
+        ixy="-1.00565663974796E-21"
+        ixz="1.3524403015242E-22"
+        iyy="1.23221647613412E-05"
+        iyz="-3.56241096455504E-11"
+        izz="1.25699738250509E-05" />
+    </inertial>
+    <visual>
+      <origin
+        xyz="0 0 0"
+        rpy="0 0 0" />
+      <geometry>
+        <mesh
+          filename="package://simpledog/meshes/lf_foot_Link.STL" />
+      </geometry>
+      <material
+        name="">
+        <color
+          rgba="0.298039215686275 0.298039215686275 0.298039215686275 1" />
+      </material>
+    </visual>
+    <collision>
+      <origin
+        xyz="0 0 0"
+        rpy="0 0 0" />
+      <geometry>
+        <mesh
+          filename="package://simpledog/meshes/lf_foot_Link.STL" />
+      </geometry>
+    </collision>
+  </link>
+  <joint
+    name="lf_foot_joint"
+    type="fixed">
+    <origin
+      xyz="0.250003601978058 0 -0.0149398452771417"
+      rpy="0 0 0" />
+    <parent
+      link="front_left_3_Link" />
+    <child
+      link="lf_foot_Link" />
+    <axis
+      xyz="0 0 0" />
+  </joint>
+  <link
+    name="front_right_1_Link">
+    <inertial>
+      <origin
+        xyz="9.7104E-17 0.012793 1.6653E-16"
+        rpy="0 0 0" />
+      <mass
+        value="1.1709" />
+      <inertia
+        ixx="0.001719"
+        ixy="-5.88E-19"
+        ixz="-1.7779E-19"
+        iyy="0.0013167"
+        iyz="-2.0543E-19"
+        izz="0.0021511" />
+    </inertial>
+    <visual>
+      <origin
+        xyz="0 0 0"
+        rpy="0 0 0" />
+      <geometry>
+        <mesh
+          filename="package://simpledog/meshes/front_right_1_Link.STL" />
+      </geometry>
+      <material
+        name="">
+        <color
+          rgba="0.89804 0.91765 0.92941 1" />
+      </material>
+    </visual>
+    <collision>
+      <origin
+        xyz="0 0 0"
+        rpy="0 0 0" />
+      <geometry>
+        <mesh
+          filename="package://simpledog/meshes/front_right_1_Link.STL" />
+      </geometry>
+    </collision>
+  </link>
+  <joint
+    name="front_right_1_joint"
+    type="revolute">
+    <origin
+      xyz="0.4 -0.175 0"
+      rpy="1.5708 1.5708 -1.5708" />
+    <parent
+      link="base_link" />
+    <child
+      link="front_right_1_Link" />
+    <axis
+      xyz="0 0 1" />
+      <limit
+      effort="100"
+      velocity="10"
+      lower="-3.0"
+      upper="3.0"/>
+  </joint>
+  <link
+    name="front_right_2_Link">
+    <inertial>
+      <origin
+        xyz="0.11432 -5.5511E-17 0.05942"
+        rpy="0 0 0" />
+      <mass
+        value="1.3902" />
+      <inertia
+        ixx="0.0030209"
+        ixy="-4.0905E-18"
+        ixz="-8.1586E-10"
+        iyy="0.026875"
+        iyz="2.3399E-19"
+        izz="0.028484" />
+    </inertial>
+    <visual>
+      <origin
+        xyz="0 0 0"
+        rpy="0 0 0" />
+      <geometry>
+        <mesh
+          filename="package://simpledog/meshes/front_right_2_Link.STL" />
+      </geometry>
+      <material
+        name="">
+        <color
+          rgba="0.89804 0.91765 0.92941 1" />
+      </material>
+    </visual>
+    <collision>
+      <origin
+        xyz="0 0 0"
+        rpy="0 0 0" />
+      <geometry>
+        <mesh
+          filename="package://simpledog/meshes/front_right_2_Link.STL" />
+      </geometry>
+    </collision>
+  </link>
+  <joint
+    name="front_right_2_joint"
+    type="revolute">
+    <origin
+      xyz="0 0 0"
+      rpy="-1.5708 0 0" />
+    <parent
+      link="front_right_1_Link" />
+    <child
+      link="front_right_2_Link" />
+    <axis
+      xyz="0 0 1" />
+      <limit
+      effort="100"
+      velocity="10"
+      lower="-3.0"
+      upper="3.0"/>
+  </joint>
+  <link
+    name="front_right_3_Link">
+    <inertial>
+      <origin
+        xyz="0.087821 6.7221E-06 -0.016729"
+        rpy="0 0 0" />
+      <mass
+        value="1.3523" />
+      <inertia
+        ixx="0.00053022"
+        ixy="-9.5809E-07"
         ixz="-0.00020532"
         iyy="0.0091429"
-        iyz="-9.1579E-07"
-        izz="0.00053022" />
-    </inertial>
-    <visual>
-      <origin
-        xyz="0 0 0"
-        rpy="0 0 0" />
-      <geometry>
-        <mesh
-          filename="package://simpledog/meshes/front_left_3_Link.STL" />
-      </geometry>
-      <material
-        name="">
-        <color
-          rgba="0.89804 0.91765 0.92941 1" />
-      </material>
-    </visual>
-    <collision>
-      <origin
-        xyz="0 0 0"
-        rpy="0 0 0" />
-      <geometry>
-        <mesh
-          filename="package://simpledog/meshes/front_left_3_Link.STL" />
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
Commit message: fix contact information

File: simpleDog/urdf/simpledog.urdf.xacro (robot description, xacro)
@@ -132,4 +132,5 @@
       lower="-3.0"
       upper="3.0"/>
+      <dynamics damping="0.7"/>
   </joint>
   <link
@@ -190,4 +191,5 @@
       lower="-3.0"
       upper="3.0"/>
+      <dynamics damping="0.7"/>
   </joint>
   <link
@@ -248,4 +250,5 @@
       lower="-3.0"
       upper="3.0"/>
+      <dynamics damping="0.7"/>
   </joint>
   <link
@@ -359,4 +362,5 @@
       lower="-3.0"
       upper="3.0"/>
+      <dynamics damping="0.7"/>
   </joint>
   <link
@@ -417,4 +421,5 @@
       lower="-3.0"
       upper="3.0"/>
+      <dynamics damping="0.7"/>
   </joint>
   <link
@@ -475,4 +480,5 @@
       lower="-3.0"
       upper="3.0"/>
+      <dynamics damping="0.7"/>
   </joint>
   <link
@@ -586,4 +592,5 @@
       lower="-3.0"
       upper="3.0"/>
+      <dynamics damping="0.7"/>
   </joint>
   <link
@@ -644,4 +651,5 @@
       lower="-3.0"
       upper="3.0"/>
+      <dynamics damping="0.7"/>
   </joint>
   <link
@@ -702,4 +710,5 @@
       lower="-3.0"
       upper="3.0"/>
+      <dynamics damping="0.7"/>
   </joint>
   <link
@@ -813,4 +822,5 @@
       lower="-3.0"
       upper="3.0"/>
+      <dynamics damping="0.7"/>
   </joint>
   <link
@@ -871,4 +881,5 @@
       lower="-3.0"
       upper="3.0"/>
+      <dynamics damping="0.7"/>
   </joint>
   <link
@@ -929,4 +940,5 @@
       lower="-3.0"
       upper="3.0"/>
+      <dynamics damping="0.7"/>
   </joint>
   <link
