Commit message: fix bug in contact information

File: simpleDog/urdf/foot_sensor_gazebo.urdf.xacro (robot description, xacro)
@@ -39,6 +39,7 @@
               <turnGravityOff>true</turnGravityOff>
               <selfCollide>false</selfCollide>
+              <maxContacts>1</maxContacts>
               <sensor type="contact" name="${foot_prefix}_contact_sensor">
-                <update_rate>100.0</update_rate>
+                <update_rate>1000.0</update_rate>
                 <contact>
                   <collision>${joint_prefix}Link_fixed_joint_lump__${foot_prefix}_Link_collision_1</collision>
@@ -48,5 +49,5 @@
                   <frameName>${foot_prefix}_Link</frameName>
                   <!-- <frameName>world</frameName> -->
-                  <updateRate>100.0</updateRate>
+                  <updateRate>1000.0</updateRate>
                   <bumperTopicName>${foot_prefix}_bumper</bumperTopicName>
                 </plugin>

File: simpleDog/urdf/kinect.urdf.xacro (robot description, xacro)
@@ -71,6 +71,6 @@
           <alwaysOn>true</alwaysOn>
           <updateRate>10.0</updateRate>
-          <imageTopicName>rgb/image_raw</imageTopicName>
-          <depthImageTopicName>depth/image_raw</depthImageTopicName>
+          <!-- <imageTopicName>rgb/image_raw</imageTopicName> -->
+          <!-- <depthImageTopicName>depth/image_raw</depthImageTopicName> -->
           <pointCloudTopicName>depth/points</pointCloudTopicName>
           <cameraInfoTopicName>rgb/camera_info</cameraInfoTopicName>

File: simpleDog/urdf/simpledog.urdf.xacro (robot description, xacro)
@@ -13,5 +13,5 @@
   <xacro:kinect_camera prefix="camera" robot_namespace="$(arg robot_namespace)"/>
   <joint name="kinect_frame_joint" type="fixed">
-    <origin xyz="0.3 0 0.1" rpy="0 0.18 0" />
+    <origin xyz="0.37 0 0.0" rpy="0 0.8 0" />
     <parent link="base_link"/>
     <child link="camera_link"/>
@@ -176,5 +176,5 @@
   <joint
     name="front_left_2_joint"
-    type="revolute">
+    type="continuous">
     <origin
       xyz="0 0 0"
@@ -235,5 +235,5 @@
   <joint
     name="front_left_3_joint"
-    type="revolute">
+    type="continuous">
     <origin
       xyz="0.250069171339977 0.000334332414087979 0.11441948932032"
@@ -406,5 +406,5 @@
   <joint
     name="front_right_2_joint"
-    type="revolute">
+    type="continuous">
     <origin
       xyz="0 0 0"
@@ -465,5 +465,5 @@
   <joint
     name="front_right_3_joint"
-    type="revolute">
+    type="continuous">
     <origin
       xyz="0.249999996334044 0 0.114419764295838"
@@ -636,5 +636,5 @@
   <joint
     name="rear_left_2_joint"
-    type="revolute">
+    type="continuous">
     <origin
       xyz="0 0 0"
@@ -695,5 +695,5 @@
   <joint
     name="rear_left_3_joint"
-    type="revolute">
+    type="continuous">
     <origin
       xyz="0.25 0 0.114419756285561"
@@ -866,5 +866,5 @@
   <joint
     name="rear_right_2_joint"
-    type="revolute">
+    type="continuous">
     <origin
       xyz="0 0 0"
@@ -925,5 +925,5 @@
   <joint
     name="rear_right_3_joint"
-    type="revolute">
+    type="continuous">
     <origin
       xyz="0.25010358767993 0.0001008844556592 0.114420076111023"
