Commit message: modified interia value of links

File: simpleDog/urdf/quadruped_model.urdf.xacro (robot description, xacro)
@@ -47,10 +47,10 @@
         value="27.801" />
       <inertia
-        ixx="0.263947"
-        ixy="-0.003647"
-        ixz="0.009059"
-        iyy="2.018039"
-        iyz="-0.000762"
-        izz="2.056397" />
+        ixx="0.263893"
+        ixy="0"
+        ixz="0"
+        iyy="2.018032"
+        iyz="0"
+        izz="2.056458" />
     </inertial>
     <visual>
@@ -87,10 +87,10 @@
         value="2.9231" />
       <inertia
-        ixx="0.007845"
-        ixy="-0.00025"
-        ixz="-7.8E-05"
-        iyy="0.005144"
-        iyz="0.000967"
-        izz="0.00794" />
+        ixx="0.004820"
+        ixy="0"
+        ixz="0"
+        iyy="0.007868"
+        iyz="0"
+        izz="0.008241" />
     </inertial>
     <visual>
@@ -135,5 +135,4 @@
       lower="-3.0"
       upper="3.0"/>
-    <dynamics damping="0.7"/>
   </joint>
   <link
@@ -146,10 +145,10 @@
         value="4.2164" />
       <inertia
-        ixx="0.00627"
-        ixy="-0.000181"
-        ixz="-8.8E-05"
-        iyy="0.029233"
-        iyz="9.2E-05"
-        izz="0.028163" />
+        ixx="0.006286"
+        ixy="0"
+        ixz="0"
+        iyy="0.028156"
+        iyz="0"
+        izz="0.029242" />
     </inertial>
     <visual>
@@ -194,5 +193,4 @@
       lower="-7.0"
       upper="7.0"/>
-    <dynamics damping="0.7"/>
   </joint>
   <link
@@ -205,10 +203,10 @@
         value="0.44457" />
       <inertia
-        ixx="0.000397"
-        ixy="-4E-06"
-        ixz="0.000261"
-        iyy="0.0065"
-        iyz="-2.4E-05"
-        izz="0.006214" />
+        ixx="0.000385"
+        ixy="0"
+        ixz="0"
+        iyy="0.006223"
+        iyz="0"
+        izz="0.006502" />
     </inertial>
     <visual>
@@ -253,5 +251,4 @@
       lower="-3.0"
       upper="3.0"/>
-      <dynamics damping="0.7"/>
   </joint>
   <link
@@ -264,10 +261,10 @@
         value="0.03332" />
       <inertia
-        ixx="1.9126E-05"
-        ixy="-1.1072E-18"
-        ixz="-4.1175E-20"
-        iyy="0"
-        iyz="1.5428E-10"
-        izz="1.3678E-05" />
+        ixx="0.000014"
+        ixy="0"
+        ixz="0"
+        iyy="0.000014"
+        iyz="0"
+        izz="0.000019" />
     </inertial>
     <visual>
@@ -317,10 +314,10 @@
         value="2.923111" />
       <inertia
-        ixx="0.007845"
-        ixy="0.00025"
-        ixz="-7.8E-05"
-        iyy="0.005144"
-        iyz="-0.000967"
-        izz="0.00794" />
+        ixx="0.004820"
+        ixy="0"
+        ixz="0"
+        iyy="0.007868"
+        iyz="0"
+        izz="0.008241" />
     </inertial>
     <visual>
@@ -365,5 +362,4 @@
       lower="-3.0"
       upper="3.0"/>
-    <dynamics damping="0.7"/>
   </joint>
   <link
@@ -376,10 +372,10 @@
         value="4.216358" />
       <inertia
-        ixx="0.00627"
-        ixy="-0.000181"
-        ixz="-8.8E-05"
-        iyy="0.029233"
-        iyz="9.2E-05"
-        izz="0.028163" />
+        ixx="0.006286"
+        ixy="0"
+        ixz="0"
+        iyy="0.028156"
+        iyz="0"
+        izz="0.029242" />
     </inertial>
     <visual>
@@ -424,5 +420,4 @@
       lower="-7.0"
       upper="7.0"/>
-    <dynamics damping="0.7"/>
   </joint>
   <link
@@ -435,10 +430,10 @@
         value="0.444569" />
       <inertia
-        ixx="0.000397"
-        ixy="-4E-06"
-        ixz="0.000261"
-        iyy="0.0065"
-        iyz="-2.4E-05"
-        izz="0.006214" />
+        ixx="0.000385"
+        ixy="0"
+        ixz="0"
+        iyy="0.006223"
+        iyz="0"
+        izz="0.006502" />
     </inertial>
     <visual>
@@ -483,5 +478,4 @@
       lower="-3.0"
       upper="3.0"/>
-    <dynamics damping="0.7"/>
   </joint>
   <link
@@ -494,10 +488,10 @@
         value="0.03332" />
       <inertia
-        ixx="1.9126E-05"
-        ixy="-1.0162E-18"
-        ixz="-1.1377E-19"
-        iyy="1.3677E-05"
-        iyz="-6.5798E-11"
-        izz="1.3678E-05" />
+        ixx="0.000014"
+        ixy="0"
+        ixz="0"
+        iyy="0.000014"
+        iyz="0"
+        izz="0.000019" />
     </inertial>
     <visual>
@@ -526,5 +520,5 @@
   </link>
   <joint
-    name="rf_foot_Link"
+    name="rf_foot_joint"
     type="fixed">
     <origin
@@ -547,10 +541,10 @@
         value="2.9231" />
       <inertia
-        ixx="0.007845"
-        ixy="0.0025"
-        ixz="-7.8E-05"
-        iyy="0.005144"
-        iyz="-0.000967"
-        izz="0.00794" />
+        ixx="0.004820"
+        ixy="0"
+        ixz="0"
+        iyy="0.007868"
+        iyz="0"
+        izz="0.008241" />
     </inertial>
     <visual>
@@ -595,5 +589,4 @@
       lower="-3.0"
       upper="3.0"/>
-    <dynamics damping="0.7"/>
   </joint>
   <link
@@ -606,10 +599,10 @@
         value="4.216358" />
       <inertia
-        ixx="0.00627"
-        ixy="-0.000181"
-        ixz="-8.8E-05"
-        iyy="0.029233"
-        iyz="9.2E-05"
-        izz="0.028163" />
+        ixx="0.006286"
+        ixy="0"
+        ixz="0"
+        iyy="0.028156"
+        iyz="0"
+        izz="0.029242" />
     </inertial>
     <visual>
@@ -654,5 +647,4 @@
       lower="-7.0"
       upper="7.0"/>
-    <dynamics damping="0.7"/>
   </joint>
   <link
@@ -665,10 +657,10 @@
         value="0.444569" />
       <inertia
-        ixx="0.000397"
-        ixy="-4E-06"
-        ixz="-0.000261"
-        iyy="0.0065"
-        iyz="-2.4E-05"
-        izz="0.006214" />
+        ixx="0.000385"
+        ixy="0"
+        ixz="0"
+        iyy="0.006223"
+        iyz="0"
+        izz="0.006502" />
     </inertial>
     <visual>
@@ -713,5 +705,4 @@
       lower="-3.0"
       upper="3.0"/>
-    <dynamics damping="0.7"/>
   </joint>
   <link
@@ -724,10 +715,10 @@
         value="0.03332" />
       <inertia
-        ixx="1.9126E-05"
-        ixy="-9.3607E-19"
-        ixz="2.2915E-19"
-        iyy="1.3677E-05"
-        iyz="-2.7943E-10"
-        izz="1.3678E-05" />
+        ixx="0.000014"
+        ixy="0"
+        ixz="0"
+        iyy="0.000014"
+        iyz="0"
+        izz="0.000019" />
     </inertial>
     <visual>
@@ -777,10 +768,10 @@
         value="2.923111" />
       <inertia
-        ixx="0.007845"
-        ixy="-0.00025"
-        ixz="7.8E-05"
-        iyy="0.005144"
-        iyz="0.000967"
-        izz="0.00794" />
+        ixx="0.004820"
+        ixy="0"
+        ixz="0"
+        iyy="0.007868"
+        iyz="0"
+        izz="0.008241" />
     </inertial>
     <visual>
@@ -825,5 +816,4 @@
       lower="-3.0"
       upper="3.0"/>
-    <dynamics damping="0.7"/>
   </joint>
   <link
@@ -836,10 +826,10 @@
         value="4.216358" />
       <inertia
-        ixx="0.00627"
-        ixy="-0.000181"
-        ixz="-8.8E-05"
-        iyy="0.029233"
-        iyz="9.2E-05"
-        izz="0.028163" />
+        ixx="0.006286"
+        ixy="0"
+        ixz="0"
+        iyy="0.028156"
+        iyz="0"
+        izz="0.029242" />
     </inertial>
     <visual>
@@ -884,5 +874,4 @@
       lower="-7.0"
       upper="7.0"/>
-    <dynamics damping="0.7"/>
   </joint>
   <link
@@ -895,10 +884,10 @@
         value="0.444569" />
       <inertia
-        ixx="0.000397"
-        ixy="-4E-06"
-        ixz="0.000261"
-        iyy="0.0065"
-        iyz="-2.4E-05"
-        izz="0.006214" />
+        ixx="0.000385"
+        ixy="0"
+        ixz="0"
+        iyy="0.006223"
+        iyz="0"
+        izz="0.006502"/>
     </inertial>
     <visual>
@@ -943,5 +932,4 @@
       lower="-3.0"
       upper="3.0"/>
-    <dynamics damping="0.7"/>
   </joint>
   <link
@@ -954,10 +942,10 @@
         value="0.03332" />
       <inertia
-        ixx="1.9126E-05"
-        ixy="-9.5089E-19"
-        ixz="6.7668E-20"
-        iyy="1.3677E-05"
-        iyz="-2.7242E-10"
-        izz="1.3678E-05" />
+        ixx="0.000014"
+        ixy="0"
+        ixz="0"
+        iyy="0.000014"
+        iyz="0"
+        izz="0.000019" />
     </inertial>
     <visual>
