Commit message: modified by yc

File: simpledog/urdf/kinect.urdf.xacro (robot description, xacro)
@@ -84,5 +84,5 @@
           <distortion_t2>0.0</distortion_t2>
           <pointCloudCutoff>0.4</pointCloudCutoff>
-          <robotNamespace>${robot_namespace}</robotNamespace>
+          <!--<robotNamespace>${robot_namespace}</robotNamespace>-->
         </plugin>
       </sensor>

File: simpledog/urdf/quadruped_model.urdf.xacro (robot description, xacro)
@@ -4,14 +4,43 @@
      For more information, please see http://wiki.ros.org/sw_urdf_exporter -->
 <robot name="quadruped_model" xmlns:xacro="http://ros.org/wiki/xacro">
-  <xacro:arg name="laser_visual"  default="false"/>
-  <xacro:arg name="camera_visual" default="false"/>
-  <xacro:arg name="imu_visual"    default="false"/>
-  <xacro:arg name="kinect_enabled"    default="true"/>
+    <xacro:include filename="$(find velodyne_description)/urdf/VLP-16.urdf.xacro"/>
+    <VLP-16 parent="base_link" name="velodyne" topic="/velodyne_points" >
+        <origin xyz="0.26  0  0.118" rpy="0 0 0" />
+    </VLP-16>
+    <link name="imu_link">
+      <inertial>
+        <mass value="0.1"/>
+        <origin rpy="0 0 0" xyz="0 0 0"/>
+        <inertia ixx="0.0001" ixy="0" ixz="0" iyy="0.000001" iyz="0" izz="0.0001"/>
+      </inertial>
+      <visual>
+        <origin rpy="0 0 0" xyz="0 0 0"/>
+        <geometry>
+          <box size="0.06 0.06 0.02"/>
+        </geometry>
+      </visual>
+      <collision>
+        <origin rpy="0 0 0" xyz="0 0 0"/>
+        <geometry>
+          <box size="0.06 0.06 0.02"/>
+        </geometry>
+      </collision>
+    </link>
+    <joint name="imu_joint" type="fixed">
+        <axis xyz="0 0 0"/>  <!--0 1 0 -->
+        <origin xyz="0.13 0 0.12" rpy="0 0 0"/>
+        <parent link="base_link"/>
+        <child link="imu_link"/>
+    </joint>
+  <!-- <xacro:arg name="laser_visual"  default="false"/> -->
+  <!-- <xacro:arg name="camera_visual" default="false"/> -->
+  <!-- <xacro:arg name="imu_visual"    default="false"/> -->
+  <xacro:arg name="kinect_enabled"    default="false"/>
     <xacro:include filename="$(find simpledog)/urdf/simpledog_gazebo.urdf.xacro" />
     <xacro:include filename="$(find simpledog)/urdf/joint_gazebo.urdf.xacro" />
-    <xacro:include filename="$(find simpledog)/urdf/kinect.urdf.xacro"/>
+    <!-- <xacro:include filename="$(find simpledog)/urdf/kinect.urdf.xacro"/> -->
     <xacro:include filename="$(find simpledog)/urdf/foot_sensor_gazebo.urdf.xacro" />
   <!--load kinect urdf-->
-  <xacro:if value="$(arg kinect_enabled)">
+<!--   <xacro:if value="$(arg kinect_enabled)">
     <xacro:kinect_camera prefix="camera" robot_namespace="$(arg robot_namespace)"/>
     <joint name="kinect_frame_joint" type="fixed">
@@ -21,4 +50,5 @@
     </joint>
   </xacro:if>
+ -->
   <!-- simple dog joints macros configure the joint driver and param-->
   <xacro:simpledog_joint joint_prefix="front_left_1_"> </xacro:simpledog_joint>

File: simpledog/urdf/simpledog_gazebo.urdf.xacro (robot description, xacro)
@@ -1,7 +1,7 @@
 <?xml version="1.0"?>
 <robot name="simpledog_gazebo" xmlns:xacro="http://ros.org/wiki/xacro">
-  <xacro:arg name="laser_visual"  default="false"/>
-  <xacro:arg name="camera_visual" default="false"/>
-  <xacro:arg name="imu_visual"    default="false"/>
+  <!-- <xacro:arg name="laser_visual"  default="false"/> -->
+  <!-- <xacro:arg name="camera_visual" default="false"/> -->
+  <!-- <xacro:arg name="imu_visual"    default="false"/> -->
   <xacro:arg name="robot_namespace" default="/simpledog" />
 <gazebo reference="base_link">
@@ -21,4 +21,44 @@
   </plugin>
 </gazebo>
+ <gazebo reference="imu_link">
+    <gravity>true</gravity>
+    <sensor name="imu" type="imu">`
+      <always_on>true</always_on>
+      <update_rate>200</update_rate>
+      <visualize>true</visualize>
+      <topic>__default_topic__</topic>
+      <plugin filename="libgazebo_ros_imu_sensor.so" name="imu_plugin">
+        <topicName>imu</topicName>
+        <bodyName>imu_link</bodyName>
+        <updateRateHZ>200.0</updateRateHZ>
+        <gaussianNoise>1e-06</gaussianNoise>
+        <xyzOffset>0 0 0</xyzOffset>
+        <rpyOffset>0 0 0</rpyOffset>
+        <frameName>imu_link</frameName>
+      </plugin>
+      <pose>0 0 0 0 0 0</pose>
+    </sensor>
+    <material>Gazebo/Blue</material>
+  </gazebo>
+  <gazebo reference="imu_link">
+    <gravity>true</gravity>
+    <sensor name="imu" type="imu">`
+      <always_on>true</always_on>
+      <update_rate>400</update_rate>
+      <visualize>true</visualize>
+      <topic>__default_topic__</topic>
+      <plugin filename="libgazebo_ros_imu_sensor.so" name="imu_plugin">
+        <topicName>imu</topicName>
+        <bodyName>imu_link</bodyName>
+        <updateRateHZ>10.0</updateRateHZ>
+        <gaussianNoise>1e-06</gaussianNoise>
+        <xyzOffset>0 0 0</xyzOffset>
+        <rpyOffset>0 0 0</rpyOffset>
+        <frameName>imu_link</frameName>
+      </plugin>
+      <pose>0 0 0 0 0 0</pose>
+    </sensor>
+    <material>Gazebo/Blue</material>
+  </gazebo>
 <!-- <gazebo reference="imu_link">
     <sensor type="imu" name="imu">
