Commit message: update simple dog launch file and do some test on urdf

File: simpledog/urdf/joint_gazebo.urdf.xacro (robot description, xacro)
@@ -47,6 +47,6 @@
                         <joint name="${joint_prefix}joint">
                                 <hardwareInterface>hardware_interface/EffortJointInterface</hardwareInterface>
-                                <!-- <hardwareInterface>hardware_interface/PositionJointInterface</hardwareInterface> -->
-                                <!-- <hardwareInterface>hardware_interface/VelocityJointInterface</hardwareInterface> -->
+                                <hardwareInterface>hardware_interface/PositionJointInterface</hardwareInterface>
+                                <hardwareInterface>hardware_interface/VelocityJointInterface</hardwareInterface>
                         </joint>
                 </transmission>

File: simpledog/urdf/quadruped_model.urdf.xacro (robot description, xacro)
@@ -33,4 +33,11 @@
         <child link="imu_link"/>
     </joint>
+    <!-- <link name = "world"/>
+    <joint name="body_link" type="fixed">
+      <parent link="world"/>
+      <child link="base_link"/>
+      <origin xyz="0 0 0" rpy="0 0 0" />
+      <axis xyz="0 0 1" />
+    </joint> -->
   <!-- <xacro:arg name="laser_visual"  default="false"/> -->
   <!-- <xacro:arg name="camera_visual" default="false"/> -->
@@ -160,5 +167,5 @@
       xyz="0 0 1" />
       <limit
-      effort="60"
+      effort="300"
       velocity="10"
       lower="-3.0"
@@ -218,5 +225,5 @@
       xyz="0 0 1" />
       <limit
-      effort="60"
+      effort="300"
       velocity="10"
       lower="-7.0"
@@ -276,5 +283,5 @@
       xyz="0 0 1" />
       <limit
-      effort="60"
+      effort="300"
       velocity="10"
       lower="-3.0"
@@ -387,5 +394,5 @@
       xyz="0 0 1" />
       <limit
-      effort="60"
+      effort="300"
       velocity="10"
       lower="-3.0"
@@ -445,5 +452,5 @@
       xyz="0 0 1" />
       <limit
-      effort="60"
+      effort="300"
       velocity="10"
       lower="-7.0"
@@ -503,5 +510,5 @@
       xyz="0 0 1" />
       <limit
-      effort="60"
+      effort="300"
       velocity="10"
       lower="-3.0"
@@ -614,5 +621,5 @@
       xyz="0 0 1" />
       <limit
-      effort="60"
+      effort="300"
       velocity="10"
       lower="-3.0"
@@ -672,5 +679,5 @@
       xyz="0 0 1" />
       <limit
-      effort="60"
+      effort="300"
       velocity="10"
       lower="-7.0"
@@ -730,5 +737,5 @@
       xyz="0 0 1" />
       <limit
-      effort="60"
+      effort="300"
       velocity="10"
       lower="-3.0"
@@ -841,5 +848,5 @@
       xyz="0 0 1" />
       <limit
-      effort="60"
+      effort="300"
       velocity="10"
       lower="-3.0"
@@ -899,5 +906,5 @@
       xyz="0 0 1" />
       <limit
-      effort="60"
+      effort="300"
       velocity="10"
       lower="-7.0"
@@ -957,5 +964,5 @@
       xyz="0 0 1" />
       <limit
-      effort="60"
+      effort="300"
       velocity="10"
       lower="-3.0"

Commit message: correct the mistakes in simple dog

File: simpledog/urdf/joint_gazebo.urdf.xacro (robot description, xacro)
@@ -47,6 +47,6 @@
                         <joint name="${joint_prefix}joint">
                                 <hardwareInterface>hardware_interface/EffortJointInterface</hardwareInterface>
-                                <hardwareInterface>hardware_interface/PositionJointInterface</hardwareInterface>
-                                <hardwareInterface>hardware_interface/VelocityJointInterface</hardwareInterface>
+                                <!-- <hardwareInterface>hardware_interface/PositionJointInterface</hardwareInterface> -->
+                                <!-- <hardwareInterface>hardware_interface/VelocityJointInterface</hardwareInterface> -->
                         </joint>
                 </transmission>

File: simpledog/urdf/quadruped_model.urdf.xacro (robot description, xacro)
@@ -43,18 +43,26 @@
   <!-- <xacro:arg name="camera_visual" default="false"/> -->
   <!-- <xacro:arg name="imu_visual"    default="false"/> -->
-  <xacro:arg name="kinect_enabled"    default="true"/>
+  <!-- <xacro:arg name="kinect_enabled"    default="true"/> -->
     <xacro:include filename="$(find simpledog)/urdf/simpledog_gazebo.urdf.xacro" />
     <xacro:include filename="$(find simpledog)/urdf/joint_gazebo.urdf.xacro" />
-    <xacro:include filename="$(find simpledog)/urdf/kinect.urdf.xacro"/>
+    <!-- <xacro:include filename="$(find simpledog)/urdf/kinect.urdf.xacro"/> -->
     <xacro:include filename="$(find simpledog)/urdf/foot_sensor_gazebo.urdf.xacro" />
-  <!--load kinect urdf-->
-  <xacro:if value="$(arg kinect_enabled)">
-    <xacro:kinect_camera prefix="camera" robot_namespace="$(arg robot_namespace)"/>
-    <joint name="kinect_frame_joint" type="fixed">
-      <origin xyz="0.5 0.0 0.0" rpy="0 0.8 0" />
-      <parent link="base_link"/>
-      <child link="camera_link"/>
-    </joint>
-  </xacro:if>
+    <!--load kinect urdf-->
+    <!-- <xacro:if value="$(arg kinect_enabled)">
+      <xacro:kinect_camera prefix="camera" robot_namespace="$(arg robot_namespace)"/>
+      <joint name="kinect_frame_joint" type="fixed">
+        <origin xyz="0.5 0 0.075" rpy="0 0.8 0" />
+        <parent link="base_link"/>
+        <child link="camera_link"/>
+      </joint>
+    </xacro:if> -->
+  <link name="zed_base_link">
+    <origin xyz="0 0 0" rpy="0 0 0"/>
+  </link>
+  <joint name="zed_base_joint" type="fixed">
+    <origin xyz="0.48 0.0 0.15" rpy="0 0.8 0" />
+    <parent link="base_link"/>
+    <child link="zed_base_link"/>
+  </joint>
   <!-- simple dog joints macros configure the joint driver and param-->
   <xacro:simpledog_joint joint_prefix="front_left_1_"> </xacro:simpledog_joint>
@@ -81,5 +89,5 @@
         rpy="0 0 0" />
       <mass
-        value="27.801" />
+        value="37.801" />
       <inertia
         ixx="0.263893"
@@ -167,5 +175,5 @@
       xyz="0 0 1" />
       <limit
-      effort="300"
+      effort="60"
       velocity="10"
       lower="-3.0"
@@ -225,5 +233,5 @@
       xyz="0 0 1" />
       <limit
-      effort="300"
+      effort="60"
       velocity="10"
       lower="-7.0"
@@ -283,5 +291,5 @@
       xyz="0 0 1" />
       <limit
-      effort="300"
+      effort="60"
       velocity="10"
       lower="-3.0"
@@ -394,5 +402,5 @@
       xyz="0 0 1" />
       <limit
-      effort="300"
+      effort="60"
       velocity="10"
       lower="-3.0"
@@ -452,5 +460,5 @@
       xyz="0 0 1" />
       <limit
-      effort="300"
+      effort="60"
       velocity="10"
       lower="-7.0"
@@ -510,5 +518,5 @@
       xyz="0 0 1" />
       <limit
-      effort="300"
+      effort="60"
       velocity="10"
       lower="-3.0"
@@ -621,5 +629,5 @@
       xyz="0 0 1" />
       <limit
-      effort="300"
+      effort="60"
       velocity="10"
       lower="-3.0"
@@ -679,5 +687,5 @@
       xyz="0 0 1" />
       <limit
-      effort="300"
+      effort="60"
       velocity="10"
       lower="-7.0"
@@ -737,5 +745,5 @@
       xyz="0 0 1" />
       <limit
-      effort="300"
+      effort="60"
       velocity="10"
       lower="-3.0"
@@ -848,5 +856,5 @@
       xyz="0 0 1" />
       <limit
-      effort="300"
+      effort="60"
       velocity="10"
       lower="-3.0"
@@ -906,5 +914,5 @@
       xyz="0 0 1" />
       <limit
-      effort="300"
+      effort="60"
       velocity="10"
       lower="-7.0"
@@ -964,5 +972,5 @@
       xyz="0 0 1" />
       <limit
-      effort="300"
+      effort="60"
       velocity="10"
       lower="-3.0"
