Commit message: some parameters adapt to real robot

File: simpledog/urdf/quadruped_model.urdf.xacro (robot description, xacro)
@@ -36,11 +36,11 @@
   <!-- <xacro:arg name="camera_visual" default="false"/> -->
   <!-- <xacro:arg name="imu_visual"    default="false"/> -->
-  <xacro:arg name="kinect_enabled"    default="false"/>
+  <xacro:arg name="kinect_enabled"    default="true"/>
     <xacro:include filename="$(find simpledog)/urdf/simpledog_gazebo.urdf.xacro" />
     <xacro:include filename="$(find simpledog)/urdf/joint_gazebo.urdf.xacro" />
-    <!-- <xacro:include filename="$(find simpledog)/urdf/kinect.urdf.xacro"/> -->
+    <xacro:include filename="$(find simpledog)/urdf/kinect.urdf.xacro"/>
     <xacro:include filename="$(find simpledog)/urdf/foot_sensor_gazebo.urdf.xacro" />
   <!--load kinect urdf-->
-<!--   <xacro:if value="$(arg kinect_enabled)">
+  <xacro:if value="$(arg kinect_enabled)">
     <xacro:kinect_camera prefix="camera" robot_namespace="$(arg robot_namespace)"/>
     <joint name="kinect_frame_joint" type="fixed">
@@ -50,5 +50,4 @@
     </joint>
   </xacro:if>
- -->
   <!-- simple dog joints macros configure the joint driver and param-->
   <xacro:simpledog_joint joint_prefix="front_left_1_"> </xacro:simpledog_joint>
@@ -161,5 +160,5 @@
       xyz="0 0 1" />
       <limit
-      effort="300"
+      effort="60"
       velocity="10"
       lower="-3.0"
@@ -219,5 +218,5 @@
       xyz="0 0 1" />
       <limit
-      effort="300"
+      effort="60"
       velocity="10"
       lower="-7.0"
@@ -277,5 +276,5 @@
       xyz="0 0 1" />
       <limit
-      effort="300"
+      effort="60"
       velocity="10"
       lower="-3.0"
@@ -388,5 +387,5 @@
       xyz="0 0 1" />
       <limit
-      effort="300"
+      effort="60"
       velocity="10"
       lower="-3.0"
@@ -446,5 +445,5 @@
       xyz="0 0 1" />
       <limit
-      effort="300"
+      effort="60"
       velocity="10"
       lower="-7.0"
@@ -504,5 +503,5 @@
       xyz="0 0 1" />
       <limit
-      effort="300"
+      effort="60"
       velocity="10"
       lower="-3.0"
@@ -563,4 +562,231 @@
   </joint>
   <link
+    name="rear_right_1_Link">
+    <inertial>
+      <origin
+        xyz="0.000688 0.104882 0.003776"
+        rpy="0 0 0" />
+      <mass
+        value="2.923111" />
+      <inertia
+        ixx="0.004820"
+        ixy="0"
+        ixz="0"
+        iyy="0.007868"
+        iyz="0"
+        izz="0.008241" />
+    </inertial>
+    <visual>
+      <origin
+        xyz="0 0 0"
+        rpy="0 0 0" />
+      <geometry>
+        <mesh
+          filename="package://simpledog/meshes/quadruped/Origin_rear_right_1_link.STL" />
+      </geometry>
+      <material
+        name="">
+        <color
+          rgba="0.79216 0.81961 0.93333 1" />
+      </material>
+    </visual>
+    <collision>
+      <origin
+        xyz="0 0 0"
+        rpy="0 0 0" />
+      <geometry>
+        <mesh
+          filename="package://simpledog/meshes/quadruped/Origin_rear_right_1_link.STL" />
+      </geometry>
+    </collision>
+  </link>
+  <joint
+    name="rear_right_1_joint"
+    type="revolute">
+    <origin
+      xyz="-0.427 -0.075 -0.0095"
+      rpy="3.1416 1.5708 0" />
+    <parent
+      link="base_link" />
+    <child
+      link="rear_right_1_Link" />
+    <axis
+      xyz="0 0 1" />
+      <limit
+      effort="60"
+      velocity="10"
+      lower="-3.0"
+      upper="3.0"/>
+  </joint>
+  <link
+    name="rear_right_2_Link">
+    <inertial>
+      <origin
+        xyz="0.184747 3.2E-05 0.129056"
+        rpy="0 0 0" />
+      <mass
+        value="4.216358" />
+      <inertia
+        ixx="0.006286"
+        ixy="0"
+        ixz="0"
+        iyy="0.028156"
+        iyz="0"
+        izz="0.029242" />
+    </inertial>
+    <visual>
+      <origin
+        xyz="0 0 0"
+        rpy="0 0 0" />
+      <geometry>
+        <mesh
+          filename="package://simpledog/meshes/quadruped/Origin_rear_right_2_link.STL" />
+      </geometry>
+      <material
+        name="">
+        <color
+          rgba="0.79216 0.81961 0.93333 1" />
+      </material>
+    </visual>
+    <collision>
+      <origin
+        xyz="0 0 0"
+        rpy="0 0 0" />
+      <geometry>
+        <mesh
+          filename="package://simpledog/meshes/quadruped/Origin_rear_right_2_link.STL" />
+      </geometry>
+    </collision>
+  </link>
+  <joint
+    name="rear_right_2_joint"
+    type="continuous">
+    <origin
+      xyz="0 0 0"
+      rpy="-1.5708 0 0" />
+    <parent
+      link="rear_right_1_Link" />
+    <child
+      link="rear_right_2_Link" />
+    <axis
+      xyz="0 0 1" />
+      <limit
+      effort="60"
+      velocity="10"
+      lower="-7.0"
+      upper="7.0"/>
+  </joint>
+  <link
+    name="rear_right_3_Link">
+    <inertial>
+      <origin
+        xyz="0.202313 0.000199 0.225432"
+        rpy="0 0 0" />
+      <mass
+        value="0.444569" />
+      <inertia
+        ixx="0.000385"
+        ixy="0"
+        ixz="0"
+        iyy="0.006223"
+        iyz="0"
+        izz="0.006502"/>
+    </inertial>
+    <visual>
+      <origin
+        xyz="0 0 0"
+        rpy="0 0 0" />
+      <geometry>
+        <mesh
+          filename="package://simpledog/meshes/quadruped/Origin_rear_right_3_link.STL" />
+      </geometry>
+      <material
+        name="">
+        <color
+          rgba="0.79216 0.81961 0.93333 1" />
+      </material>
+    </visual>
+    <collision>
+      <origin
+        xyz="0 0 0"
+        rpy="0 0 0" />
+      <geometry>
+        <mesh
+          filename="package://simpledog/meshes/quadruped/Origin_rear_right_3_link.STL" />
+      </geometry>
+    </collision>
+  </link>
+  <joint
+    name="rear_right_3_joint"
+    type="continuous">
+    <origin
+      xyz="0.308 0 0"
+      rpy="0 0 0" />
+    <parent
+      link="rear_right_2_Link" />
+    <child
+      link="rear_right_3_Link" />
+    <axis
+      xyz="0 0 1" />
+      <limit
+      effort="60"
+      velocity="10"
+      lower="-3.0"
+      upper="3.0"/>
+  </joint>
+  <link
+    name="rh_foot_Link">
+    <inertial>
+      <origin
+        xyz="0.022126 -1.6187E-13 -1E-06"
+        rpy="0 0 0" />
+      <mass
+        value="0.03332" />
+      <inertia
+        ixx="0.000014"
+        ixy="0"
+        ixz="0"
+        iyy="0.000014"
+        iyz="0"
+        izz="0.000019" />
+    </inertial>
+    <visual>
+      <origin
+        xyz="0 0 0"
+        rpy="0 0 0" />
+      <geometry>
+        <mesh
+          filename="package://simpledog/meshes/quadruped/Origin_rr_foot_link.STL" />
+      </geometry>
+      <material
+        name="">
+        <color
+          rgba="0 0 0 1" />
+      </material>
+    </visual>
+    <collision>
+      <origin
+        xyz="0 0 0"
+        rpy="0 0 0" />
+      <geometry>
+        <mesh
+          filename="package://simpledog/meshes/quadruped/Origin_rr_foot_link.STL" />
+      </geometry>
+    </collision>
+  </link>
+  <joint
+    name="rh_foot_joint"
+    type="fixed">
+    <origin
+      xyz="0.308 0 0.22053"
+      rpy="0 0 0" />
+    <parent
+      link="rear_right_3_Link" />
+    <child
+      link="rh_foot_Link" />
+    <axis
+      xyz="0 0 0" />
+  </joint>
+  <link
     name="rear_left_1_Link">
     <inertial>
@@ -615,5 +841,5 @@
       xyz="0 0 1" />
       <limit
-      effort="300"
+      effort="60"
       velocity="10"
       lower="-3.0"
@@ -673,5 +899,5 @@
       xyz="0 0 1" />
       <limit
-      effort="300"
+      effort="60"
       velocity="10"
       lower="-7.0"
@@ -731,5 +957,5 @@
       xyz="0 0 1" />
       <limit
-      effort="300"
+      effort="60"
       velocity="10"
       lower="-3.0"
@@ -789,230 +1015,3 @@
       xyz="0 0 0" />
   </joint>
-  <link
-    name="rear_right_1_Link">
-    <inertial>
-      <origin
-        xyz="0.000688 0.104882 0.003776"
-        rpy="0 0 0" />
-      <mass
-        value="2.923111" />
-      <inertia
-        ixx="0.004820"
-        ixy="0"
-        ixz="0"
-        iyy="0.007868"
-        iyz="0"
-        izz="0.008241" />
-    </inertial>
-    <visual>
-      <origin
-        xyz="0 0 0"
-        rpy="0 0 0" />
-      <geometry>
-        <mesh
-          filename="package://simpledog/meshes/quadruped/Origin_rear_right_1_link.STL" />
-      </geometry>
-      <material
-        name="">
-        <color
-          rgba="0.79216 0.81961 0.93333 1" />
-      </material>
-    </visual>
-    <collision>
-      <origin
-        xyz="0 0 0"
-        rpy="0 0 0" />
-      <geometry>
-        <mesh
-          filename="package://simpledog/meshes/quadruped/Origin_rear_right_1_link.STL" />
-      </geometry>
-    </collision>
-  </link>
-  <joint
-    name="rear_right_1_joint"
-    type="revolute">
-    <origin
-      xyz="-0.427 -0.075 -0.0095"
-      rpy="3.1416 1.5708 0" />
-    <parent
-      link="base_link" />
-    <child
-      link="rear_right_1_Link" />
-    <axis
-      xyz="0 0 1" />
-      <limit
-      effort="300"
-      velocity="10"
-      lower="-3.0"
-      upper="3.0"/>
-  </joint>
-  <link
-    name="rear_right_2_Link">
-    <inertial>
-      <origin
-        xyz="0.184747 3.2E-05 0.129056"
-        rpy="0 0 0" />
-      <mass
-        value="4.216358" />
-      <inertia
-        ixx="0.006286"
-        ixy="0"
-        ixz="0"
-        iyy="0.028156"
-        iyz="0"
-        izz="0.029242" />
-    </inertial>
-    <visual>
-      <origin
-        xyz="0 0 0"
-        rpy="0 0 0" />
-      <geometry>
-        <mesh
-          filename="package://simpledog/meshes/quadruped/Origin_rear_right_2_link.STL" />
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
Commit message: add ZED in URDF

File: simpledog/urdf/quadruped_model.urdf.xacro (robot description, xacro)
@@ -36,18 +36,23 @@
   <!-- <xacro:arg name="camera_visual" default="false"/> -->
   <!-- <xacro:arg name="imu_visual"    default="false"/> -->
-  <xacro:arg name="kinect_enabled"    default="true"/>
+  <!-- <xacro:arg name="kinect_enabled"    default="true"/> -->
     <xacro:include filename="$(find simpledog)/urdf/simpledog_gazebo.urdf.xacro" />
     <xacro:include filename="$(find simpledog)/urdf/joint_gazebo.urdf.xacro" />
-    <xacro:include filename="$(find simpledog)/urdf/kinect.urdf.xacro"/>
+    <!-- <xacro:include filename="$(find simpledog)/urdf/kinect.urdf.xacro"/> -->
     <xacro:include filename="$(find simpledog)/urdf/foot_sensor_gazebo.urdf.xacro" />
   <!--load kinect urdf-->
-  <xacro:if value="$(arg kinect_enabled)">
+  <!-- <xacro:if value="$(arg kinect_enabled)">
     <xacro:kinect_camera prefix="camera" robot_namespace="$(arg robot_namespace)"/>
     <joint name="kinect_frame_joint" type="fixed">
       <origin xyz="0.5 0.0 0.0" rpy="0 0.8 0" />
       <parent link="base_link"/>
-      <child link="camera_link"/>
+      <child link="zed_base_link"/>
     </joint>
-  </xacro:if>
+  </xacro:if> -->
+  <joint name="zed_base_joint" type="fixed">
+    <origin xyz="0.5 0.0 0.0" rpy="0 0.8 0" />
+    <parent link="base_link"/>
+    <child link="zed_base_link"/>
+  </joint>
   <!-- simple dog joints macros configure the joint driver and param-->
   <xacro:simpledog_joint joint_prefix="front_left_1_"> </xacro:simpledog_joint>

Commit message: add ZED in URDF

File: simpledog/urdf/quadruped_model.urdf.xacro (robot description, xacro)
@@ -41,13 +41,7 @@
     <!-- <xacro:include filename="$(find simpledog)/urdf/kinect.urdf.xacro"/> -->
     <xacro:include filename="$(find simpledog)/urdf/foot_sensor_gazebo.urdf.xacro" />
-  <!--load kinect urdf-->
-  <!-- <xacro:if value="$(arg kinect_enabled)">
-    <xacro:kinect_camera prefix="camera" robot_namespace="$(arg robot_namespace)"/>
-    <joint name="kinect_frame_joint" type="fixed">
-      <origin xyz="0.5 0.0 0.0" rpy="0 0.8 0" />
-      <parent link="base_link"/>
-      <child link="zed_base_link"/>
-    </joint>
-  </xacro:if> -->
+  <link name="zed_base_link">
+    <origin xyz="0 0 0" rpy="0 0 0"/>
+  </link>
   <joint name="zed_base_joint" type="fixed">
     <origin xyz="0.5 0.0 0.0" rpy="0 0.8 0" />

Commit message: modified ZED TF in URDF

File: simpledog/urdf/quadruped_model.urdf.xacro (robot description, xacro)
@@ -45,5 +45,5 @@
   </link>
   <joint name="zed_base_joint" type="fixed">
-    <origin xyz="0.5 0.0 0.0" rpy="0 0.8 0" />
+    <origin xyz="0.5 0.0 0.15" rpy="0 0.8 0" />
     <parent link="base_link"/>
     <child link="zed_base_link"/>

Commit message: final commit by WSHY

File: simpledog/urdf/quadruped_model.urdf.xacro (robot description, xacro)
@@ -33,4 +33,11 @@
         <child link="imu_link"/>
     </joint>
+    <link name = "world"/>
+    <joint name="body_link" type="fixed">
+      <parent link="world"/>
+      <child link="base_link"/>
+      <origin xyz="0 0 0" rpy="0 0 0" />
+      <axis xyz="0 0 1" />
+    </joint>
   <!-- <xacro:arg name="laser_visual"  default="false"/> -->
   <!-- <xacro:arg name="camera_visual" default="false"/> -->
@@ -41,9 +48,18 @@
     <!-- <xacro:include filename="$(find simpledog)/urdf/kinect.urdf.xacro"/> -->
     <xacro:include filename="$(find simpledog)/urdf/foot_sensor_gazebo.urdf.xacro" />
+    <!--load kinect urdf-->
+    <!-- <xacro:if value="$(arg kinect_enabled)">
+      <xacro:kinect_camera prefix="camera" robot_namespace="$(arg robot_namespace)"/>
+      <joint name="kinect_frame_joint" type="fixed">
+        <origin xyz="0.5 0 0.075" rpy="0 0.8 0" />
+        <parent link="base_link"/>
+        <child link="camera_link"/>
+      </joint>
+    </xacro:if> -->
   <link name="zed_base_link">
     <origin xyz="0 0 0" rpy="0 0 0"/>
   </link>
   <joint name="zed_base_joint" type="fixed">
-    <origin xyz="0.5 0.0 0.15" rpy="0 0.8 0" />
+    <origin xyz="0.48 0.0 0.15" rpy="0 0.8 0" />
     <parent link="base_link"/>
     <child link="zed_base_link"/>
@@ -73,5 +89,5 @@
         rpy="0 0 0" />
       <mass
-        value="27.801" />
+        value="37.801" />
       <inertia
         ixx="0.263893"

Commit message: final commit by WSHY

File: simpledog/urdf/quadruped_model.urdf.xacro (robot description, xacro)
@@ -33,4 +33,11 @@
         <child link="imu_link"/>
     </joint>
+    <!-- <link name = "world"/>
+    <joint name="body_link" type="fixed">
+      <parent link="world"/>
+      <child link="base_link"/>
+      <origin xyz="0 0 0" rpy="0 0 0" />
+      <axis xyz="0 0 1" />
+    </joint> -->
   <!-- <xacro:arg name="laser_visual"  default="false"/> -->
   <!-- <xacro:arg name="camera_visual" default="false"/> -->
@@ -41,9 +48,18 @@
     <!-- <xacro:include filename="$(find simpledog)/urdf/kinect.urdf.xacro"/> -->
     <xacro:include filename="$(find simpledog)/urdf/foot_sensor_gazebo.urdf.xacro" />
+    <!--load kinect urdf-->
+    <!-- <xacro:if value="$(arg kinect_enabled)">
+      <xacro:kinect_camera prefix="camera" robot_namespace="$(arg robot_namespace)"/>
+      <joint name="kinect_frame_joint" type="fixed">
+        <origin xyz="0.5 0 0.075" rpy="0 0.8 0" />
+        <parent link="base_link"/>
+        <child link="camera_link"/>
+      </joint>
+    </xacro:if> -->
   <link name="zed_base_link">
     <origin xyz="0 0 0" rpy="0 0 0"/>
   </link>
   <joint name="zed_base_joint" type="fixed">
-    <origin xyz="0.5 0.0 0.15" rpy="0 0.8 0" />
+    <origin xyz="0.48 0.0 0.15" rpy="0 0.8 0" />
     <parent link="base_link"/>
     <child link="zed_base_link"/>
@@ -73,5 +89,5 @@
         rpy="0 0 0" />
       <mass
-        value="27.801" />
+        value="37.801" />
       <inertia
         ixx="0.263893"

Commit message: test configure controller

File: simpledog/urdf/quadruped_model.urdf.xacro (robot description, xacro)
@@ -33,5 +33,5 @@
         <child link="imu_link"/>
     </joint>
-    <link name = "world"/>
+   <!-- <link name = "world"/>
     <joint name="body_link" type="fixed">
       <parent link="world"/>
@@ -39,5 +39,5 @@
       <origin xyz="0 0 0" rpy="0 0 0" />
       <axis xyz="0 0 1" />
-    </joint>
+    </joint> -->
   <!-- <xacro:arg name="laser_visual"  default="false"/> -->
   <!-- <xacro:arg name="camera_visual" default="false"/> -->
